File: LVDS_RasPi_Hat.kicad_sch (KiCad schematic)
At the start: 1 part, among them J1 Raspberry_Pi_2_3

Commit message: v2
Connections:
- net NIM0: now also J1.36 (GPIO16); no longer J1.27 (ID_SD/GPIO0)
- net NIM1: now also J1.27 (ID_SD/GPIO0); no longer J1.24 (~{CE0}/GPIO8)
- net NIM2: now also J1.24 (~{CE0}/GPIO8); no longer J1.36 (GPIO16)
- net TRIGGER0 renamed CONFIG2
- net TRIGGER1 renamed CONFIG15
- net TRIGGER10 renamed CONFIG10
- net TRIGGER11 renamed CONFIG6
- net TRIGGER12 renamed CONFIG11
- net TRIGGER13 renamed CONFIG13
- net TRIGGER14 renamed CONFIG14
- net TRIGGER15 renamed CONFIG7
- net TRIGGER2 renamed CONFIG4
- net TRIGGER3 renamed CONFIG5
- net TRIGGER4 renamed CONFIG3
- net TRIGGER5 renamed CONFIG1
- net TRIGGER6 renamed CONFIG8
- net TRIGGER7 renamed CONFIG12
- net TRIGGER8 renamed CONFIG9
- net TRIGGER9 renamed CONFIG0
- net TS_BUS_SEL0 renamed TS_BUS_SEL
- net TS_BUS_SEL1: no longer names the net of J1.5 (SCL/GPIO3)
- net TS_BUS_SEL2: no longer names the net of J1.7 (GCLK0/GPIO4)
- net TS_BUS_SEL3: no longer names the net of J1.11 (GPIO17)
- no-connect marks 0 -> 3
Other:
- added sheet Configuration and Indication (configuration.kicad_sch)
- sheet Trigger Interface ports: added TS_BUS_SEL; removed TRIGGER[0..15], TS_BUS_SEL[0..3]
- company: MIT Physics -> MIT
