File: trigger_interface.kicad_sch (KiCad schematic)
At the start: 27 parts, among them J2 RJHSE508002, J3 Conn_Coaxial_Small, J4 Conn_Coaxial_Small, J5 Conn_Coaxial_Small, J6 Conn_Coaxial_Small, U1 SN65MLVD206BD, U2 SN65MLVD206BD, U3 SN65MLVD206BD, U4 SN65MLVD206BD, U5 SN65LVDT348D

Commit message: v2
Parts:
- removed C5: C100n, Capacitor_SMD:C_0402_1005Metric_Pad0.74x0.62mm_HandSolder, symbol Device:C
- removed J3, J5: Conn_Coaxial_Small, Connector_Coaxial:SMA_Amphenol_901-143_Horizontal, symbol Connector:Conn_Coaxial_Small
- removed J4, J6: Conn_Coaxial_Small, EPL_00_250_NTN:CONN_EPK.00.250.NTN_LMO, symbol Connector:Conn_Coaxial_Small
- removed JP1, JP2, JP3, JP4: SolderJumper_2_Open, Jumper:SolderJumper-2_P1.3mm_Open_RoundedPad1.0x1.5mm, symbol Jumper:SolderJumper_2_Open
- removed R1, R2, R3, R4: R100, Resistor_SMD:R_0402_1005Metric_Pad0.72x0.64mm_HandSolder, symbol Device:R
- removed R5, R6, R7, R8: R50, Resistor_SMD:R_0402_1005Metric_Pad0.72x0.64mm_HandSolder, symbol Device:R
- removed U5: SN65LVDT348D, SN65LVDT348D:D16-M, symbol SN65LVDT348D:SN65LVDT348D
- added C1: C100n, Capacitor_SMD:C_0402_1005Metric_Pad0.74x0.62mm_HandSolder, symbol Device:C
- added U1: SN65LVDT348D, SN65LVDT348D:D16, symbol SN65LVDT348D:SN65LVDT348D
- renumbered C1 to C2, C2 to C3, C3 to C4, C4 to C5, U1 to U2, U2 to U3, U3 to U4, U4 to U5
Connections:
- net TS_BUS_SEL1 is gone; now on net TS_BUS_SEL: U3.2 (RE_N), U3.3 (DE)
- net TS_BUS_SEL2 is gone; now on net TS_BUS_SEL: U4.2 (RE_N), U4.3 (DE)
- net TS_BUS_SEL3 is gone; now on net TS_BUS_SEL: U5.2 (RE_N), U5.3 (DE)
- net +3V3: now also C1.1, U1.13 (VCC), U1.16 (EN)
- net D1+: no longer J2.2_1
- net D1-: no longer J2.2_2
- net D2+: no longer J2.2_3
- net D2-: no longer J2.2_6
- net D3+: no longer J2.2_5
- net D3-: no longer J2.2_4
- net D4+: no longer J2.2_7
- net D4-: no longer J2.2_8
- net GND: now also C1.2, U1.12 (GND), U1.9 (*EN)
- net TS_BUS0 renamed D0
- net TS_BUS1 renamed D1
- net TS_BUS2 renamed D2
- net TS_BUS3 renamed D3
- net TS_BUS_SEL0 renamed TS_BUS_SEL
- new net S0: U1.10 (ROUT4)
- new net S1: U1.11 (ROUT3)
- new net S1+: J2.2_2, U1.7 (RIN4+)
- new net S1-: J2.2_1, U1.8
- new net S2: U1.14 (ROUT2)
- new net S2+: J2.2_6, U1.6 (RIN3+)
- new net S2-: J2.2_3, U1.5
- new net S3: U1.15 (ROUT1)
- new net S3+: J2.2_4, U1.3 (RIN2+)
- new net S3-: J2.2_5, U1.4
- new net S4+: J2.2_8, U1.2 (RIN1+)
- new net S4-: J2.2_7, U1.1
Other:
- removed sheet Trigger Signals
- company: MIT Physics -> MIT
- moved on the sheet: C2, C3, C4, C5
